Commit message: Se actualizó el tutorial y se terminó era_description hasta antes de usar MoveIt setup Assistant

File: src/era_description/urdf/era_description.urdf (robot description, URDF)
Before this commit: robot era_description, 8 links, 7 joints
Links:
- added link world
Joints:
- added joint base_joint: type fixed, parent world, child base_link, origin xyz=0.0 0.0 0.17 rpy=0 0 0

Commit message: Se añadió el paquete era_moveit_config y se actualizó algunas cosas del tutorial

File: src/era_description/urdf/era_description.urdf (robot description, URDF)
Before this commit: robot era_description, 9 links, 8 joints
Joints:
- removed joint base_joint
- added joint joint_0: type fixed, parent world, child link_0, origin xyz=0.0 0.0 0.17 rpy=0 0 0
